File: VPThermo.brd (EAGLE design)
At the start: 54 x 64 mm, 54 parts, among them SW1 SPST_TACT-KMR2, SW2 SPST_TACT-KMR2, U1 REG1117, U2 ESP-12F, U3 MCP41010-I/SN, U4 RT6208GE, U5 SN74LVC1G3157DBVR, X1 5 x Screw clamp

Commit message: Revision C
Parts:
- removed R6: 10k, eagle-ltspice:R0603
- added C16: 100n, rcl:C0603
- added D2: S1M, diode:SMA
- added U6: MCP130, ola-microchip:SOT23
- C11: value 10u -> 22u
- C7: value 150p -> 22u; device rcl:C0603 -> resistor:C0805
- L1: value SDR0302-121KL -> ME3220-153KLB
- R1: value 127k -> 56k
- R11: value 24k -> 10k
- R15: value 1k -> 10k
- R7: value 6k8 -> 270k
- U4: value RT6208GE -> LMR14206; device richtek:SOT-23-6 -> ola_texas:SOT-23-6
- moved R11 8.25 mm to (2.50, 8.00), turned to 90 degrees
- moved R1 6.52 mm to (2.50, 12.5), turned to 90 degrees
- moved L1 6.40 mm to (6.00, 16.0)
- moved TP5 4.03 mm to (11.5, 25.0)
- moved C7 2.06 mm to (10.0, 19.0), turned to 0 degrees
- moved C10 1.58 mm to (9.00, 5.00)
- moved U4 1.50 mm to (6.00, 9.00), turned to 270 degrees
- moved C11 1.41 mm to (10.0, 16.5), turned to 0 degrees
- moved C14 1.12 mm to (11.5, 5.00)
- moved C5 1.00 mm to (13.0, 50.0)
- moved C8 0.71 mm to (14.0, 5.00)
- moved C13 0.50 mm to (16.5, 5.00)
- moved R15 0.50 mm to (13.0, 47.5)
- renumbered R13 to FB1, R14 to FB2
Connections:
- removed net N$8: C5.2, R15.1, R6.1, SW1.2, SW1.4, TP6.TP, U2.GPIO16, U2.RESET
- new net N$22: SW1.2, SW1.4, TP6.TP, U2.GPIO16, U2.RESET, U6.1
- new net N$23: C16.1, D2.C, L1.1, U4.6
- net +3V3: now also C5.1, R15.1, U6.2; no longer R6.2
- net GND: now also C5.2, C7.2, D2.A, U6.3; no longer C5.1
- net N$14: now also U4.4
- net N$19: now also U4.3; no longer C7.2, U4.1
- net N$3: now also C16.2, U4.1; no longer L1.1, U4.6
Routing:
- net N$8: track 41.7 -> 0.00 mm, vias 2 -> 0
- net N$22: track 0.00 -> 30.7 mm, vias 0 -> 2
- net N$23: track 0.00 -> 12.4 mm
- net +5V: track 66.7 -> 74.6 mm
- net +3V3: track 121.7 -> 114.6 mm
- net N$19: track 8.58 -> 5.33 mm
- net N$3: track 3.24 -> 2.24 mm
- net GND: vias 64 -> 68
Other:
- board text added: "PCB201701C"
- board text removed: "PCB201701B"
